File: Hardware/Production/SparkFun_MicroMod_Function_Board_Blues_Notecarrier-Panel.brd (EAGLE design)
At the start: 133.6 x 149.6 mm, 576 parts, among them J13 NOTECARD, J14 MICROMOD_FUNCTION_STANDARD, J18 NOTECARD, J19 MICROMOD_FUNCTION_STANDARD, J2 MICROMOD_FUNCTION_STANDARD, J23 NOTECARD, J24 MICROMOD_FUNCTION_STANDARD, J28 NOTECARD, J29 MICROMOD_FUNCTION_STANDARD, J6 NOTECARD, J8 NOTECARD, J9 MICROMOD_FUNCTION_STANDARD, Q1 220mA/50V/3.5Ω, Q10 20V/4.2A/52mΩ/1.4W, Q11 220mA/50V/3.5Ω, Q12 20V/4.2A/52mΩ/1.4W, Q13 220mA/50V/3.5Ω, Q14 220mA/50V/3.5Ω, Q15 20V/4.2A/52mΩ/1.4W, Q16 20V/4.2A/52mΩ/1.4W, Q17 220mA/50V/3.5Ω, Q18 20V/4.2A/52mΩ/1.4W, Q19 220mA/50V/3.5Ω, Q2 20V/4.2A/52mΩ/1.4W, Q20 220mA/50V/3.5Ω, Q21 20V/4.2A/52mΩ/1.4W, Q22 20V/4.2A/52mΩ/1.4W, Q23 220mA/50V/3.5Ω, Q24 20V/4.2A/52mΩ/1.4W, Q25 220mA/50V/3.5Ω, Q26 220mA/50V/3.5Ω, Q27 20V/4.2A/52mΩ/1.4W, Q28 20V/4.2A/52mΩ/1.4W, Q29 220mA/50V/3.5Ω, Q3 220mA/50V/3.5Ω, Q30 20V/4.2A/52mΩ/1.4W, Q31 220mA/50V/3.5Ω, Q32 220mA/50V/3.5Ω, Q33 20V/4.2A/52mΩ/1.4W, Q34 20V/4.2A/52mΩ/1.4W, Q35 220mA/50V/3.5Ω, Q36 20V/4.2A/52mΩ/1.4W, Q4 20V/4.2A/52mΩ/1.4W, Q5 220mA/50V/3.5Ω, Q6 20V/4.2A/52mΩ/1.4W, Q7 220mA/50V/3.5Ω, Q8 220mA/50V/3.5Ω, Q9 20V/4.2A/52mΩ/1.4W, U1 EEPROM, U10 TCR2EF33, U11 EEPROM, U12 TCR2EF33, U2 TCR2EF33, U3 EEPROM, U4 TCR2EF33, U5 EEPROM, U6 TCR2EF33, U7 EEPROM, U8 TCR2EF33, U9 EEPROM

Commit message: Rev v11
AEN wasn't enabled by default because it was missing a passive. Added passive and rerouted.
Parts:
- removed Q31, Q32, Q35: 220mA/50V/3.5Ω, SparkFun-DiscreteSemi:SOT23-3
- removed Q33, Q34, Q36: 20V/4.2A/52mΩ/1.4W, SparkFun-DiscreteSemi:SOT23-3
- removed R100: 1, SparkFun-Resistors:0603
- removed R101, R97: 10k, SparkFun-Resistors:0402-TIGHT
- removed R102, R98, R99: 100, SparkFun-Resistors:0402-TIGHT
- Q12, Q16, Q21, Q22, Q27: value 20V/4.2A/52mΩ/1.4W -> 220mA/50V/3.5Ω
- Q13, Q14, Q19, Q20, Q23, Q25, Q29, Q8: value 220mA/50V/3.5Ω -> 20V/4.2A/52mΩ/1.4W
- R17, R48, R51, R64, R65, R68, R81, R85: value 100 -> 10k
- R18, R50: value 10k -> 560Ω
- R19, R36, R53: value 560Ω -> 10k
- R22, R38, R39, R54, R55, R71, R86: value 10k -> 5.1k
- R24, R40, R41, R57: value 5.1k -> 1k
- R26, R42: value 1k -> 2.2k
- R27: value 2.2k -> 2.2M
- R28, R96: value 2.2M -> 10k
- R29, R46: value 10k -> 100
- R31, R47: value 100 -> 1; device SparkFun-Resistors:0402-TIGHT -> SparkFun-Resistors:0603
- R32, R49, R83: value 1 -> 10k; device SparkFun-Resistors:0603 -> SparkFun-Resistors:0402-TIGHT
- R34, R82: value 100 -> 560Ω
- R43, R59: value 1k -> 2.2M
- R44: value 2.2k -> 10k
- R45, R62: value 2.2M -> 100
- R56, R72, R73, R88, R89: value 10k -> 1k
- R58, R74: value 5.1k -> 2.2k
- R60, R76: value 1k -> 10k
- R61, R78: value 2.2k -> 100
- R63: value 10k -> 1; device SparkFun-Resistors:0402-TIGHT -> SparkFun-Resistors:0603
- R66: value 1 -> 560Ω; device SparkFun-Resistors:0603 -> SparkFun-Resistors:0402-TIGHT
- R70, R87: value 560Ω -> 5.1k
- R75, R91: value 5.1k -> 2.2M
- R77, R93, R94: value 1k -> 100
- R79: value 2.2M -> 1; device SparkFun-Resistors:0402-TIGHT -> SparkFun-Resistors:0603
- R90: value 10k -> 2.2k
- R92: value 5.1k -> 10k
- R95: value 2.2k -> 1; device SparkFun-Resistors:0402-TIGHT -> SparkFun-Resistors:0603
- moved R49 142.3 mm to (4.89, 122.8)
- moved Q16 142.1 mm to (16.2, 128.2), turned to 90 degrees
- moved R50 115.3 mm to (8.89, 127.8), turned to 90 degrees
- moved R51 113.1 mm to (10.3, 127.8), turned to 270 degrees
- moved Q18 109.7 mm to (12.8, 127.2), turned to 180 degrees
- moved Q17 108.6 mm to (23.2, 128.2)
- moved R17 72.8 mm to (70.6, 13.5)
- moved R34 70.9 mm to (104.6, 8.55), turned to 270 degrees
- moved R33 70.7 mm to (108.6, 13.5)
- moved Q5 62.9 mm to (59.3, 8.10), turned to 270 degrees
- moved Q11 62.9 mm to (97.3, 8.10), turned to 270 degrees
- moved Q12 58.9 mm to (90.3, 8.10), turned to 270 degrees
- moved R93 56.5 mm to (90.2, 130.3)
- moved R72 55.7 mm to (60.9, 74.5)
- moved R56 54.9 mm to (22.9, 74.5)
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Connections:
- removed net AUX_PWR: J2.55, Q5.1
- removed net AUX_PWR1: J9.55, Q11.1
- removed net AUX_PWR2: J14.55, Q17.1
- removed net AUX_PWR3: J19.55, Q23.1
- removed net AUX_PWR4: J24.55, Q29.1
- removed net AUX_PWR5: J29.55, Q35.1
- removed net N$101 (its old number): Q26.3, R82.1
- removed net N$109 (its old number): J26.B5, R91.2
- removed net N$114 (its old number): PWR_LED5.2, R94.1
- removed net N$115: R93.1, VIO_LED5.2
- removed net N$116: D56.C, R95.2
- removed net N$117: AUX_EN_LED5.2, R95.1
- removed net N$118: R97.1, U12.3
- removed net N$120: D58.A, Q33.3
- removed net N$121: Q31.3, R98.1
- removed net N$122: Q32.3, R99.1
- removed net N$123: MEAS5.2, MEAS5.4, R100.1
- removed net N$125: Q36.1, R101.1, R102.2
- removed net N$126: Q35.3, R102.1
- removed net N$21 (its old number): J9.71, R19.2
- removed net N$24 (its old number): J4.B5, R23.2
- removed net N$32 (its old number): AUX_EN_LED1.2, R27.1
- removed net N$35 (its old number): D18.A, Q9.3
- removed net N$38 (its old number): Q8.3, R31.1
- removed net N$44 (its old number): Q15.1, R38.1, R47.2
- removed net N$52 (its old number): R42.1, VIO_LED2.2
- removed net N$57 (its old number): D28.A, Q15.3
- removed net N$63 (its old number): Q17.3, R51.1
- removed net N$71 (its old number): D35.C, R60.2
- removed net N$76 (its old number): R63.1, U8.3
- removed net N$95 (its old number): D46.C, R78.2
- new net !AUX_PWR!: J2.55, Q6.1, R10.2
- new net !AUX_PWR!1: J9.55, Q10.1, R32.2
- new net !AUX_PWR!2: J14.55, Q15.1, R48.2
- new net !AUX_PWR!3: J19.55, Q20.1, R64.2
- new net !AUX_PWR!4: J24.55, Q25.1, R80.2
- new net !AUX_PWR!5: J29.55, Q30.1, R96.2
- new net N$103: D55.C, R89.2
- new net N$111: Q26.3, R93.1
- new net N$22: J4.B5, R22.2
- new net N$26: D15.C, R25.2
- new net N$34: Q5.3, R29.1
- new net N$36: MEAS1.2, MEAS1.4, R31.1
- new net N$40: Q13.1, R36.1, R45.2
- new net N$48: R40.1, VIO_LED2.2
- new net N$56: MEAS2.2, MEAS2.4, R47.1
- new net N$61: J16.B5, R54.2
- new net N$69: AUX_EN_LED3.2, R58.1
- new net N$77: J24.71, R66.2
- new net N$98: Q29.1, R85.1, R94.2
- net 3.3V: no longer R10.2
- net 3.3V1: now also Q10.2, R17.1; no longer Q12.2, R18.1, R33.2
- net 3.3V2: now also Q15.2, R33.1; no longer Q18.2, R35.1, R50.2
- net 3.3V3: now also Q20.2, R49.1; no longer Q24.2, R52.1, R67.2
- net 3.3V4: now also Q25.2, R65.1; no longer Q30.2, R69.1, R84.2
- net 3.3V5: now also Q30.2, R81.1; no longer Q36.2, R101.2, R86.1
- net 3V3_IN1: now also Q8.2, R19.1, R20.2; no longer Q9.2, R20.1, R21.2
- net 3V3_IN2: now also Q13.2, R35.1, R36.2; no longer Q15.2, R37.1, R38.2
- net 3V3_IN3: now also Q18.2, R51.1, R52.2; no longer Q21.2, R54.1, R55.2
- net 3V3_IN4: now also Q23.2, R67.1, R68.2; no longer Q27.2, R71.1, R72.2
- net 3V3_IN5: now also Q28.2, R83.1, R84.2; no longer Q33.2, R88.1, R89.2
- net AUX_EN1: now also Q10.3; no longer Q12.3
- net AUX_EN2: now also Q15.3; no longer Q18.3
- net AUX_EN3: now also Q20.3; no longer Q24.3
- net AUX_EN4: now also Q25.3; no longer Q30.3
- net AUX_EN5: now also Q30.3; no longer Q36.3
- net EWP1: now also R17.2; no longer R18.2
- net EWP2: now also R33.2; no longer R35.2
- net EWP3: now also R49.2; no longer R52.2
- net EWP4: now also R65.2; no longer R69.2
- net EWP5: now also R81.2; no longer R86.2
- net GND: now also R10.1; no longer Q5.2
- net GND1: now also Q5.2, R22.1, R27.1, R32.1; no longer Q11.2, Q8.2, R24.1, R28.1
- net GND2: now also Q11.2, Q12.2, R38.1, R39.1, R43.1, R48.1; no longer Q13.2, Q14.2, Q17.2, R40.1, R41.1, R45.1
- net GND3: now also Q16.2, Q17.2, R54.1, R55.1, R59.1, R64.1; no longer Q19.2, Q20.2, Q23.2, R57.1, R58.1, R62.1
- net GND4: now also Q21.2, Q22.2, R70.1, R71.1, R80.1; no longer Q25.2, Q26.2, Q29.2, R74.1, R79.1
- net GND5: now also Q26.2, Q27.2, R86.1, R87.1; no longer Q31.2, Q32.2, Q35.2, R92.1
- net N$100: now also J26.A5, R87.2; no longer Q25.3, R81.1
- net N$102: now also D54.C, R88.2; no longer MEAS4.2, MEAS4.4, R83.1
- net N$104: now also PWR_LED5.2, R89.1; no longer Q30.1, R84.1, R85.2
- net N$105: now also R88.1, VIO_LED5.2; no longer Q29.3, R85.1
- net N$106: now also D56.C, R90.2; no longer J29.71, R87.2
- net N$107: now also AUX_EN_LED5.2, R90.1; no longer Q33.1, R89.1, R98.2
- net N$108: now also R92.1, U12.3; no longer Q34.1, R90.1, R99.2
- net N$110: now also D58.A, Q28.3; no longer J26.A5, R92.2
- net N$112: now also Q27.3, R94.1; no longer D54.C, R93.2
- net N$113: now also MEAS5.2, MEAS5.4, R95.1; no longer D55.C, R94.2
- net N$19: now also J9.71, R18.2; no longer Q6.1, R10.1, R17.2
- net N$20: now also Q8.1, R20.1, R29.2; no longer Q5.3, R17.1
- net N$23: now also J4.A5, R23.2; no longer Q10.1, R22.1, R31.2
- net N$25: now also D14.C; no longer J4.A5
- net N$27: now also PWR_LED1.2, R25.1; no longer D14.C, R25.2
- net N$28: now also R24.1, VIO_LED1.2; no longer D15.C, R26.2
- net N$29: now also D16.C, R26.2; no longer PWR_LED1.2, R26.1
- net N$30: now also AUX_EN_LED1.2, R26.1; no longer R25.1, VIO_LED1.2
- net N$31: now also R28.1, U4.3; no longer D16.C, R27.2
- net N$33: now also D18.A, Q8.3; no longer R29.1, U4.3
- net N$39: now also J14.71, R34.2; no longer MEAS1.2, MEAS1.4, R32.1
- net N$41: now also Q14.1, R37.1, R46.2; no longer Q12.1, R33.1, R34.2
- net N$42: now also J11.B5, R38.2; no longer Q11.3, R34.1
- net N$43: now also J11.A5, R39.2; no longer J14.71, R36.2
- net N$45: now also D24.C, R40.2; no longer Q16.1, R39.1, R48.2
- net N$46: now also D25.C, R41.2; no longer J11.B5, R40.2
- net N$47: now also PWR_LED2.2, R41.1; no longer J11.A5, R41.2
- net N$49: now also D26.C; no longer D24.C
- net N$50: now also AUX_EN_LED2.2, R42.1; no longer D25.C, R43.2
- net N$51: now also R44.1, U6.3; no longer PWR_LED2.2, R43.1
- net N$53: now also D28.A, Q13.3; no longer D26.C, R44.2
- net N$54: now also Q11.3, R45.1; no longer AUX_EN_LED2.2, R44.1
- net N$55: now also Q12.3; no longer U6.3
- net N$58: now also J19.71, R50.2; no longer Q13.3, R47.1
- net N$59: now also Q18.1, R52.1, R61.2; no longer Q14.3, R48.1
- net N$60: now also Q19.1, R53.1, R62.2; no longer MEAS2.2, MEAS2.4, R49.1
- net N$62: now also J16.A5, R55.2; no longer Q18.1, R50.1, R51.2
- net N$64: now also D34.C, R56.2; no longer J19.71, R53.2
- net N$65: now also D35.C, R57.2; no longer Q21.1, R55.1, R64.2
- net N$66: now also PWR_LED3.2, R57.1; no longer Q22.1, R56.1, R65.2
- net N$67: now also R56.1, VIO_LED3.2; no longer J16.B5, R57.2
- net N$68: now also D36.C; no longer J16.A5
- net N$70: now also R60.1, U8.3; no longer D34.C, R59.2
- net N$72: now also D38.A, Q18.3; no longer PWR_LED3.2, R60.1
- net N$73: now also Q16.3, R61.1; no longer R59.1, VIO_LED3.2
- net N$74: now also Q17.3, R62.1; no longer D36.C, R61.2
- net N$75: now also MEAS3.2, MEAS3.4, R63.1; no longer AUX_EN_LED3.2, R61.1
- net N$78: now also Q23.1, R68.1, R77.2; no longer D38.A, Q21.3
- net N$79: now also Q24.1, R69.1, R78.2; no longer Q19.3, R64.1
- net N$80: now also J21.B5, R70.2; no longer Q20.3, R65.1
- net N$81: now also J21.A5, R71.2; no longer MEAS3.2, MEAS3.4, R66.1
- net N$83: now also D44.C, R72.2; no longer Q24.1, R67.1, R68.2
- net N$84: now also D45.C, R73.2; no longer Q23.3, R68.1
- net N$85: now also PWR_LED4.2, R73.1; no longer J24.71, R70.2
- net N$86: now also VIO_LED4.2; no longer Q27.1, R81.2
- net N$87: now also D46.C, R74.2; no longer Q28.1, R73.1, R82.2
- net N$88: now also AUX_EN_LED4.2, R74.1; no longer J21.B5, R74.2
- net N$89: now also R76.1, U10.3; no longer J21.A5, R75.2
- net N$91: now also D48.A, Q23.3; no longer D44.C, R76.2
- net N$92: now also Q21.3, R77.1; no longer D45.C, R77.2
- net N$93: now also Q22.3, R78.1; no longer PWR_LED4.2, R77.1
- net N$94: now also MEAS4.2, MEAS4.4, R79.1; no longer R76.1, VIO_LED4.2
- net N$96: now also J29.71, R82.2; no longer AUX_EN_LED4.2, R78.1
- net N$97: now also Q28.1, R84.1, R93.2; no longer R80.1, U10.3
- net N$99: now also J26.B5, R86.2; no longer D48.A, Q27.3
- net PWR_EN1: now also Q5.1, R18.1, R19.2; no longer Q8.1, R19.1, R20.2
- net PWR_EN2: now also Q11.1, Q12.1, R34.1, R35.2; no longer Q13.1, Q14.1, R36.1, R37.2
- net PWR_EN3: now also Q16.1, Q17.1, R50.1, R51.2; no longer Q19.1, Q20.1, R53.1, R54.2
- net PWR_EN4: now also Q21.1, Q22.1, R66.1, R67.2; no longer Q25.1, Q26.1, R70.1, R71.2
- net PWR_EN5: now also Q26.1, Q27.1, R82.1, R83.2; no longer Q31.1, Q32.1, R87.1, R88.2
- net VCC1: now also Q9.3; no longer Q10.3
- net VCC2: now also Q14.3; no longer Q16.3
- net VCC3: now also Q19.3; no longer Q22.3
- net VCC4: now also Q24.3; no longer Q28.3
- net VCC5: now also Q29.3; no longer Q34.3
- net VCC_IN1: now also Q9.2, R21.2; no longer Q10.2, R22.2
- net VCC_IN2: now also Q14.2, R37.2; no longer Q16.2, R39.2
- net VCC_IN3: now also Q19.2, R53.2; no longer Q22.2, R56.2
- net VCC_IN4: now also Q24.2, R69.2; no longer Q28.2, R73.2
- net VCC_IN5: now also Q29.2, R85.2; no longer Q34.2, R90.2
- net VIN1: now also R27.2, R31.2; no longer R29.2, R32.2
- net VIN2: now also R43.2, R44.2, R47.2; no longer R45.2, R46.2, R49.2
- net VIN3: now also R59.2, R60.2; no longer R62.2, R66.2
- net VIN4: now also R75.2, R76.2; no longer R80.2, R83.2
- net VIN5: now also R91.2, R92.2, R95.2; no longer R100.2, R96.2, R97.2
Routing:
- net !AUX_PWR!2: track 0.00 -> 52.3 mm, vias 0 -> 2
- net !AUX_PWR!1: track 0.00 -> 52.3 mm, vias 0 -> 2
- net !AUX_PWR!: track 0.00 -> 52.3 mm, vias 0 -> 2
- net !AUX_PWR!5: track 0.00 -> 52.3 mm, vias 0 -> 2
- net !AUX_PWR!4: track 0.00 -> 52.3 mm, vias 0 -> 2
- net !AUX_PWR!3: track 0.00 -> 52.3 mm, vias 0 -> 2
- net AUX_PWR5: track 48.0 -> 0.00 mm, vias 2 -> 0
- net AUX_PWR4: track 48.0 -> 0.00 mm, vias 2 -> 0
- net AUX_PWR3: track 48.0 -> 0.00 mm, vias 2 -> 0
- net AUX_PWR2: track 48.0 -> 0.00 mm, vias 2 -> 0
- net AUX_PWR1: track 48.0 -> 0.00 mm, vias 2 -> 0
- net AUX_PWR: track 48.0 -> 0.00 mm, vias 2 -> 0
- net N$21 (its old number): track 21.6 -> 0.00 mm
- net N$77: track 0.00 -> 21.6 mm
- net N$64: track 21.6 -> 1.51 mm
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Other:
- board text added: "v11"
- board text removed: "v10"
